File: keyboard2-kicad/keyboard/keyboard.kicad_pcb (KiCad board)
At the start: 2 copper layers, 0 parts

Commit message: keyb pcb finished w/ wrong switches
Parts:
- added C1: 10u, Capacitor_SMD:C_0402_1005Metric, B.Cu at (44.6, 31.6)
- added C10: 1u, Capacitor_SMD:C_0402_1005Metric, F.Cu at (60.9, 24.5)
- added C11: 1u, Capacitor_SMD:C_0402_1005Metric, F.Cu at (60.9, 25.5)
- added C12: 100n, Capacitor_SMD:C_0402_1005Metric, F.Cu at (71.3, 26.8)
- added C13: 100n, Capacitor_SMD:C_0402_1005Metric, F.Cu at (51.0, 29.4)
- added C14: 100n, Capacitor_SMD:C_0402_1005Metric, F.Cu at (55.4, 38.2)
- added C15: 15p, Capacitor_SMD:C_0402_1005Metric, F.Cu at (87.8, 20.0)
- added C16: 15p, Capacitor_SMD:C_0402_1005Metric, F.Cu at (82.5, 20.0)
- added C2: 10u, Capacitor_SMD:C_0402_1005Metric, B.Cu at (47.6, 33.1)
- added C3: 100n, Capacitor_SMD:C_0402_1005Metric, F.Cu at (63.2, 33.4)
- added C4: 100n, Capacitor_SMD:C_0402_1005Metric, F.Cu at (62.0, 35.6)
- added C5: 100n, Capacitor_SMD:C_0402_1005Metric, F.Cu at (71.6, 27.8)
- added C6: 100n, Capacitor_SMD:C_0402_1005Metric, F.Cu at (67.2, 22.0)
- added C7: 100n, Capacitor_SMD:C_0402_1005Metric, F.Cu at (63.6, 23.1)
- added C8: 100n, Capacitor_SMD:C_0402_1005Metric, F.Cu at (60.9, 23.5)
- added C9: 100n, Capacitor_SMD:C_0402_1005Metric, F.Cu at (52.3, 28.4)
- added D1: D, Diode_SMD:D_SOD-323, F.Cu at (57.0, 56.0)
- added D10: D, Diode_SMD:D_SOD-323, F.Cu at (228.0, 56.0)
- added D100: D, Diode_SMD:D_SOD-323, F.Cu at (400.0, 140.9)
- added D101: LED, LED_SMD:LED_0603_1608Metric, F.Cu at (50.2, 57.0)
- added D102: LED, LED_SMD:LED_0603_1608Metric, F.Cu at (69.2, 57.0)
- added D103: LED, LED_SMD:LED_0603_1608Metric, F.Cu at (88.2, 57.0)
- added D104: LED, LED_SMD:LED_0603_1608Metric, F.Cu at (107.2, 57.0)
- added D105: LED, LED_SMD:LED_0603_1608Metric, F.Cu at (126.2, 57.0)
- added D106: LED, LED_SMD:LED_0603_1608Metric, F.Cu at (145.2, 57.0)
- added D107: LED, LED_SMD:LED_0603_1608Metric, F.Cu at (164.2, 57.0)
- added D108: LED, LED_SMD:LED_0603_1608Metric, F.Cu at (183.2, 57.0)
- added D109: LED, LED_SMD:LED_0603_1608Metric, F.Cu at (202.2, 57.0)
- added D11: D, Diode_SMD:D_SOD-323, F.Cu at (247.0, 56.0)
- added D110: LED, LED_SMD:LED_0603_1608Metric, F.Cu at (221.2, 57.0)
- added D111: LED, LED_SMD:LED_0603_1608Metric, F.Cu at (240.2, 57.0)
- added D112: LED, LED_SMD:LED_0603_1608Metric, F.Cu at (259.2, 57.0)
- added D113: LED, LED_SMD:LED_0603_1608Metric, F.Cu at (279.0, 57.0)
- added D114: LED, LED_SMD:LED_0603_1608Metric, F.Cu at (298.0, 57.0)
- added D115: LED, LED_SMD:LED_0603_1608Metric, F.Cu at (317.1, 57.0)
- added D116: LED, LED_SMD:LED_0603_1608Metric, F.Cu at (336.1, 57.0)
- added D117: LED, LED_SMD:LED_0603_1608Metric, F.Cu at (355.1, 57.0)
- added D118: LED, LED_SMD:LED_0603_1608Metric, F.Cu at (374.2, 57.0)
- added D119: LED, LED_SMD:LED_0603_1608Metric, F.Cu at (393.2, 57.0)
- added D12: D, Diode_SMD:D_SOD-323, F.Cu at (266.0, 56.0)
- added D120: LED, LED_SMD:LED_0603_1608Metric, F.Cu at (50.2, 76.0)
- added D121: LED, LED_SMD:LED_0603_1608Metric, F.Cu at (69.0, 76.0)
- added D122: LED, LED_SMD:LED_0603_1608Metric, F.Cu at (88.2, 76.0)
- added D123: LED, LED_SMD:LED_0603_1608Metric, F.Cu at (107.2, 76.0)
- added D124: LED, LED_SMD:LED_0603_1608Metric, F.Cu at (126.2, 76.0)
- added D125: LED, LED_SMD:LED_0603_1608Metric, F.Cu at (145.2, 76.0)
- added D126: LED, LED_SMD:LED_0603_1608Metric, F.Cu at (164.0, 76.0)
- added D127: LED, LED_SMD:LED_0603_1608Metric, F.Cu at (183.2, 76.0)
- added D128: LED, LED_SMD:LED_0603_1608Metric, F.Cu at (202.0, 76.0)
- added D129: LED, LED_SMD:LED_0603_1608Metric, F.Cu at (222.2, 76.0)
- added D13: D, Diode_SMD:D_SOD-323, F.Cu at (285.0, 56.0)
- added D130: LED, LED_SMD:LED_0603_1608Metric, F.Cu at (240.2, 76.0)
- added D131: LED, LED_SMD:LED_0603_1608Metric, F.Cu at (259.2, 76.0)
- added D132: LED, LED_SMD:LED_0603_1608Metric, F.Cu at (279.4, 76.0)
- added D133: LED, LED_SMD:LED_0603_1608Metric, F.Cu at (308.0, 76.0)
- added D134: LED, LED_SMD:LED_0603_1608Metric, F.Cu at (336.2, 76.0)
- added D135: LED, LED_SMD:LED_0603_1608Metric, F.Cu at (355.0, 76.0)
- added D136: LED, LED_SMD:LED_0603_1608Metric, F.Cu at (374.0, 76.0)
- added D137: LED, LED_SMD:LED_0603_1608Metric, F.Cu at (392.2, 76.0)
- added D138: LED, LED_SMD:LED_0603_1608Metric, F.Cu at (55.0, 95.0)
- added D139: LED, LED_SMD:LED_0603_1608Metric, F.Cu at (79.2, 95.0)
- added D14: D, Diode_SMD:D_SOD-323, F.Cu at (304.0, 56.0)
- added D140: LED, LED_SMD:LED_0603_1608Metric, F.Cu at (98.2, 95.0)
- added D141: LED, LED_SMD:LED_0603_1608Metric, F.Cu at (116.8, 95.0)
- added D142: LED, LED_SMD:LED_0603_1608Metric, F.Cu at (135.8, 95.0)
- added D143: LED, LED_SMD:LED_0603_1608Metric, F.Cu at (154.8, 95.0)
- added D144: LED, LED_SMD:LED_0603_1608Metric, F.Cu at (173.2, 95.0)
- added D145: LED, LED_SMD:LED_0603_1608Metric, F.Cu at (192.2, 95.0)
- added D146: LED, LED_SMD:LED_0603_1608Metric, F.Cu at (212.2, 95.0)
- added D147: LED, LED_SMD:LED_0603_1608Metric, F.Cu at (231.2, 95.0)
- added D148: LED, LED_SMD:LED_0603_1608Metric, F.Cu at (250.2, 95.0)
- added D149: LED, LED_SMD:LED_0603_1608Metric, F.Cu at (269.0, 95.0)
- added D15: D, Diode_SMD:D_SOD-323, F.Cu at (323.0, 56.0)
- added D150: LED, LED_SMD:LED_0603_1608Metric, F.Cu at (288.0, 95.0)
- added D151: LED, LED_SMD:LED_0603_1608Metric, F.Cu at (312.0, 95.0)
- added D152: LED, LED_SMD:LED_0603_1608Metric, F.Cu at (336.2, 95.0)
- added D153: LED, LED_SMD:LED_0603_1608Metric, F.Cu at (354.8, 95.0)
- added D154: LED, LED_SMD:LED_0603_1608Metric, F.Cu at (374.2, 95.0)
- added D155: LED, LED_SMD:LED_0603_1608Metric, F.Cu at (57.2, 114.0)
- added D156: LED, LED_SMD:LED_0603_1608Metric, F.Cu at (83.2, 114.0)
- added D157: LED, LED_SMD:LED_0603_1608Metric, F.Cu at (102.2, 114.0)
- added D158: LED, LED_SMD:LED_0603_1608Metric, F.Cu at (121.2, 114.0)
- added D159: LED, LED_SMD:LED_0603_1608Metric, F.Cu at (140.2, 114.0)
- added D16: D, Diode_SMD:D_SOD-323, F.Cu at (342.0, 56.0)
- added D160: LED, LED_SMD:LED_0603_1608Metric, F.Cu at (159.2, 114.0)
- added D161: LED, LED_SMD:LED_0603_1608Metric, F.Cu at (178.2, 114.0)
- added D162: LED, LED_SMD:LED_0603_1608Metric, F.Cu at (197.2, 114.0)
- added D163: LED, LED_SMD:LED_0603_1608Metric, F.Cu at (216.2, 114.0)
- added D164: LED, LED_SMD:LED_0603_1608Metric, F.Cu at (235.2, 114.0)
- added D165: LED, LED_SMD:LED_0603_1608Metric, F.Cu at (254.2, 114.0)
- added D166: LED, LED_SMD:LED_0603_1608Metric, F.Cu at (274.2, 114.0)
- added D167: LED, LED_SMD:LED_0603_1608Metric, F.Cu at (306.2, 114.0)
- added D168: LED, LED_SMD:LED_0603_1608Metric, F.Cu at (336.2, 114.0)
- added D169: LED, LED_SMD:LED_0603_1608Metric, F.Cu at (354.8, 114.0)
- added D17: D, Diode_SMD:D_SOD-323, F.Cu at (361.0, 56.0)
- added D170: LED, LED_SMD:LED_0603_1608Metric, F.Cu at (374.0, 114.0)
- added D171: LED, LED_SMD:LED_0603_1608Metric, F.Cu at (393.2, 105.0)
- added D172: LED, LED_SMD:LED_0603_1608Metric, F.Cu at (62.2, 133.0)
- added D173: LED, LED_SMD:LED_0603_1608Metric, F.Cu at (93.2, 133.0)
- added D174: LED, LED_SMD:LED_0603_1608Metric, F.Cu at (112.2, 133.0)
- added D175: LED, LED_SMD:LED_0603_1608Metric, F.Cu at (131.2, 133.0)
- added D176: LED, LED_SMD:LED_0603_1608Metric, F.Cu at (150.2, 133.0)
- added D177: LED, LED_SMD:LED_0603_1608Metric, F.Cu at (169.2, 133.0)
- added D178: LED, LED_SMD:LED_0603_1608Metric, F.Cu at (188.2, 133.0)
- added D179: LED, LED_SMD:LED_0603_1608Metric, F.Cu at (207.2, 133.0)
- added D18: D, Diode_SMD:D_SOD-323, F.Cu at (381.0, 56.0)
- added D180: LED, LED_SMD:LED_0603_1608Metric, F.Cu at (226.2, 133.0)
- added D181: LED, LED_SMD:LED_0603_1608Metric, F.Cu at (245.2, 133.0)
- added D182: LED, LED_SMD:LED_0603_1608Metric, F.Cu at (264.2, 133.0)
- added D183: LED, LED_SMD:LED_0603_1608Metric, F.Cu at (290.2, 133.0)
- added D184: LED, LED_SMD:LED_0603_1608Metric, F.Cu at (317.0, 133.0)
- added D185: LED, LED_SMD:LED_0603_1608Metric, F.Cu at (335.2, 133.0)
- added D186: LED, LED_SMD:LED_0603_1608Metric, F.Cu at (354.2, 133.0)
- added D187: LED, LED_SMD:LED_0603_1608Metric, F.Cu at (374.0, 133.0)
- added D188: LED, LED_SMD:LED_0603_1608Metric, F.Cu at (52.0, 152.0)
- added D189: LED, LED_SMD:LED_0603_1608Metric, F.Cu at (77.0, 152.2)
- added D19: D, Diode_SMD:D_SOD-323, F.Cu at (400.0, 56.0)
- added D190: LED, LED_SMD:LED_0603_1608Metric, F.Cu at (100.0, 152.0)
- added D191: LED, LED_SMD:LED_0603_1608Metric, F.Cu at (169.8, 152.0)
- added D192: LED, LED_SMD:LED_0603_1608Metric, F.Cu at (241.0, 152.0)
- added D193: LED, LED_SMD:LED_0603_1608Metric, F.Cu at (260.2, 152.0)
- added D194: LED, LED_SMD:LED_0603_1608Metric, F.Cu at (278.2, 152.0)
- added D195: LED, LED_SMD:LED_0603_1608Metric, F.Cu at (298.2, 152.0)
- added D196: LED, LED_SMD:LED_0603_1608Metric, F.Cu at (317.0, 152.0)
- added D197: LED, LED_SMD:LED_0603_1608Metric, F.Cu at (336.2, 152.0)
- added D198: LED, LED_SMD:LED_0603_1608Metric, F.Cu at (355.2, 152.0)
- added D199: LED, LED_SMD:LED_0603_1608Metric, F.Cu at (374.2, 152.0)
- added D2: D, Diode_SMD:D_SOD-323, F.Cu at (76.0, 56.0)
- added D20: D, Diode_SMD:D_SOD-323, F.Cu at (57.0, 75.0)
- added D200: LED, LED_SMD:LED_0603_1608Metric, F.Cu at (393.2, 142.0)
- added D21: D, Diode_SMD:D_SOD-323, F.Cu at (76.0, 75.0)
- added D22: D, Diode_SMD:D_SOD-323, F.Cu at (95.0, 75.0)
- added D23: D, Diode_SMD:D_SOD-323, F.Cu at (114.0, 75.0)
- added D24: D, Diode_SMD:D_SOD-323, F.Cu at (133.0, 75.0)
- added D25: D, Diode_SMD:D_SOD-323, F.Cu at (152.0, 75.0)
- added D26: D, Diode_SMD:D_SOD-323, F.Cu at (171.0, 75.0)
- added D27: D, Diode_SMD:D_SOD-323, F.Cu at (190.0, 75.0)
- added D28: D, Diode_SMD:D_SOD-323, F.Cu at (209.0, 75.0)
- added D29: D, Diode_SMD:D_SOD-323, F.Cu at (228.0, 75.0)
- added D3: D, Diode_SMD:D_SOD-323, F.Cu at (95.0, 56.0)
- added D30: D, Diode_SMD:D_SOD-323, F.Cu at (247.0, 75.0)
- added D31: D, Diode_SMD:D_SOD-323, F.Cu at (266.0, 75.0)
- added D32: D, Diode_SMD:D_SOD-323, F.Cu at (285.0, 75.0)
- added D33: D, Diode_SMD:D_SOD-323, F.Cu at (314.0, 75.0)
- added D34: D, Diode_SMD:D_SOD-323, F.Cu at (343.0, 75.0)
- added D35: D, Diode_SMD:D_SOD-323, F.Cu at (362.0, 75.0)
- added D36: D, Diode_SMD:D_SOD-323, F.Cu at (381.0, 75.0)
- added D37: D, Diode_SMD:D_SOD-323, F.Cu at (400.0, 75.0)
- added D38: D, Diode_SMD:D_SOD-323, F.Cu at (62.0, 94.0)
- added D39: D, Diode_SMD:D_SOD-323, F.Cu at (86.0, 94.0)
- added D4: D, Diode_SMD:D_SOD-323, F.Cu at (114.0, 56.0)
- added D40: D, Diode_SMD:D_SOD-323, F.Cu at (104.0, 94.0)
- added D41: D, Diode_SMD:D_SOD-323, F.Cu at (124.0, 94.0)
- added D42: D, Diode_SMD:D_SOD-323, F.Cu at (143.0, 94.0)
- added D43: D, Diode_SMD:D_SOD-323, F.Cu at (162.0, 94.0)
- added D44: D, Diode_SMD:D_SOD-323, F.Cu at (181.0, 94.0)
- added D45: D, Diode_SMD:D_SOD-323, F.Cu at (200.0, 94.0)
- added D46: D, Diode_SMD:D_SOD-323, F.Cu at (219.0, 94.0)
- added D47: D, Diode_SMD:D_SOD-323, F.Cu at (238.0, 94.0)
- added D48: D, Diode_SMD:D_SOD-323, F.Cu at (257.0, 94.0)
- added D49: D, Diode_SMD:D_SOD-323, F.Cu at (276.0, 94.0)
- added D5: D, Diode_SMD:D_SOD-323, F.Cu at (133.0, 56.0)
- added D50: D, Diode_SMD:D_SOD-323, F.Cu at (295.0, 94.0)
- added D51: D, Diode_SMD:D_SOD-323, F.Cu at (319.0, 94.0)
- added D52: D, Diode_SMD:D_SOD-323, F.Cu at (343.0, 94.0)
- added D53: D, Diode_SMD:D_SOD-323, F.Cu at (361.0, 94.0)
- added D54: D, Diode_SMD:D_SOD-323, F.Cu at (381.0, 94.0)
- added D55: D, Diode_SMD:D_SOD-323, F.Cu at (64.0, 113.0)
- added D56: D, Diode_SMD:D_SOD-323, F.Cu at (90.0, 113.0)
- added D57: D, Diode_SMD:D_SOD-323, F.Cu at (109.0, 113.0)
- added D58: D, Diode_SMD:D_SOD-323, F.Cu at (128.0, 113.0)
- added D59: D, Diode_SMD:D_SOD-323, F.Cu at (147.0, 113.0)
- added D6: D, Diode_SMD:D_SOD-323, F.Cu at (152.0, 56.0)
- added D60: D, Diode_SMD:D_SOD-323, F.Cu at (166.0, 113.0)
- added D61: D, Diode_SMD:D_SOD-323, F.Cu at (185.0, 113.0)
- added D62: D, Diode_SMD:D_SOD-323, F.Cu at (204.0, 113.0)
- added D63: D, Diode_SMD:D_SOD-323, F.Cu at (224.0, 113.0)
- added D64: D, Diode_SMD:D_SOD-323, F.Cu at (243.0, 113.0)
- added D65: D, Diode_SMD:D_SOD-323, F.Cu at (262.0, 113.0)
- added D66: D, Diode_SMD:D_SOD-323, F.Cu at (281.0, 113.0)
- added D67: D, Diode_SMD:D_SOD-323, F.Cu at (313.0, 113.0)
- added D68: D, Diode_SMD:D_SOD-323, F.Cu at (343.0, 113.0)
- added D69: D, Diode_SMD:D_SOD-323, F.Cu at (362.0, 113.0)
- added D7: D, Diode_SMD:D_SOD-323, F.Cu at (171.0, 56.0)
- added D70: D, Diode_SMD:D_SOD-323, F.Cu at (381.0, 113.0)
- added D71: D, Diode_SMD:D_SOD-323, F.Cu at (400.0, 103.0)
- added D72: D, Diode_SMD:D_SOD-323, F.Cu at (69.0, 132.0)
- added D73: D, Diode_SMD:D_SOD-323, F.Cu at (100.0, 131.9)
- added D74: D, Diode_SMD:D_SOD-323, F.Cu at (119.0, 131.9)
- added D75: D, Diode_SMD:D_SOD-323, F.Cu at (138.0, 131.9)
- added D76: D, Diode_SMD:D_SOD-323, F.Cu at (157.0, 132.1)
- added D77: D, Diode_SMD:D_SOD-323, F.Cu at (176.0, 132.0)
- added D78: D, Diode_SMD:D_SOD-323, F.Cu at (195.0, 132.0)
- added D79: D, Diode_SMD:D_SOD-323, F.Cu at (214.0, 132.0)
- added D8: D, Diode_SMD:D_SOD-323, F.Cu at (190.0, 56.0)
- added D80: D, Diode_SMD:D_SOD-323, F.Cu at (233.0, 132.0)
- added D81: D, Diode_SMD:D_SOD-323, F.Cu at (252.0, 131.9)
- added D82: D, Diode_SMD:D_SOD-323, F.Cu at (271.0, 131.9)
- added D83: D, Diode_SMD:D_SOD-323, F.Cu at (297.0, 131.9)
- added D84: D, Diode_SMD:D_SOD-323, F.Cu at (324.0, 132.0)
- added D85: D, Diode_SMD:D_SOD-323, F.Cu at (343.0, 132.0)
- added D86: D, Diode_SMD:D_SOD-323, F.Cu at (362.0, 132.0)
- added D87: D, Diode_SMD:D_SOD-323, F.Cu at (381.0, 132.0)
- added D88: D, Diode_SMD:D_SOD-323, F.Cu at (59.0, 151.0)
- added D89: D, Diode_SMD:D_SOD-323, F.Cu at (83.0, 151.1)
- added D9: D, Diode_SMD:D_SOD-323, F.Cu at (209.0, 56.0)
- added D90: D, Diode_SMD:D_SOD-323, F.Cu at (107.0, 151.1)
- added D91: D, Diode_SMD:D_SOD-323, F.Cu at (177.0, 151.0)
- added D92: D, Diode_SMD:D_SOD-323, F.Cu at (248.0, 151.1)
- added D93: D, Diode_SMD:D_SOD-323, F.Cu at (266.0, 151.0)
- added D94: D, Diode_SMD:D_SOD-323, F.Cu at (285.0, 151.0)
- added D95: D, Diode_SMD:D_SOD-323, F.Cu at (305.0, 151.1)
- added D96: D, Diode_SMD:D_SOD-323, F.Cu at (323.0, 151.0)
- added D97: D, Diode_SMD:D_SOD-323, F.Cu at (343.0, 151.0)
- added D98: D, Diode_SMD:D_SOD-323, F.Cu at (362.0, 151.0)
- added D99: D, Diode_SMD:D_SOD-323, F.Cu at (381.0, 150.9)
- added J1: DC-005, DC-005:NINIGI_DC-005, F.Cu at (31.2, 24.8)
- added J2: TYPE-C-31-M-12, TYPE-C-31-M-12:HRO_TYPE-C-31-M-12, F.Cu at (44.0, 16.3)
- added J3: Touchscreen, Connector_PinHeader_2.54mm:PinHeader_1x14_P2.54mm_Vertical, F.Cu at (416.6, 152.0)
- added J4: Touchscreen, Connector_PinHeader_2.54mm:PinHeader_1x14_P2.54mm_Vertical, F.Cu at (416.5, 80.0)
- added M1: Motor_Servo, Connector_PinHeader_2.54mm:PinHeader_1x03_P2.54mm_Horizontal, B.Cu at (125.2, 17.0)
- added M10: Motor_Servo, Connector_PinHeader_2.54mm:PinHeader_1x03_P2.54mm_Horizontal, B.Cu at (312.8, 17.0)
- added M2: Motor_Servo, Connector_PinHeader_2.54mm:PinHeader_1x03_P2.54mm_Horizontal, B.Cu at (146.0, 17.0)
- added M3: Motor_Servo, Connector_PinHeader_2.54mm:PinHeader_1x03_P2.54mm_Horizontal, B.Cu at (166.9, 17.0)
- added M4: Motor_Servo, Connector_PinHeader_2.54mm:PinHeader_1x03_P2.54mm_Horizontal, B.Cu at (187.7, 17.0)
- added M5: Motor_Servo, Connector_PinHeader_2.54mm:PinHeader_1x03_P2.54mm_Horizontal, B.Cu at (208.6, 17.0)
- added M6: Motor_Servo, Connector_PinHeader_2.54mm:PinHeader_1x03_P2.54mm_Horizontal, B.Cu at (229.4, 17.0)
- added M7: Motor_Servo, Connector_PinHeader_2.54mm:PinHeader_1x03_P2.54mm_Horizontal, B.Cu at (250.2, 17.0)
- added M8: Motor_Servo, Connector_PinHeader_2.54mm:PinHeader_1x03_P2.54mm_Horizontal, B.Cu at (271.1, 17.0)
- added M9: Motor_Servo, Connector_PinHeader_2.54mm:PinHeader_1x03_P2.54mm_Horizontal, B.Cu at (291.9, 17.0)
- added R1: 1k, Resistor_SMD:R_0402_1005Metric, F.Cu at (83.5, 22.5)
- added R10: 680R, Resistor_SMD:R_0402_1005Metric, F.Cu at (66.5, 57.0)
- added R100: 680R, Resistor_SMD:R_0402_1005Metric, F.Cu at (238.1, 152.0)
- added R101: 680R, Resistor_SMD:R_0402_1005Metric, F.Cu at (257.3, 152.0)
- added R102: 680R, Resistor_SMD:R_0402_1005Metric, F.Cu at (275.1, 152.0)
- added R103: 680R, Resistor_SMD:R_0402_1005Metric, F.Cu at (295.5, 152.0)
- added R104: 680R, Resistor_SMD:R_0402_1005Metric, F.Cu at (314.3, 152.0)
- added R105: 680R, Resistor_SMD:R_0402_1005Metric, F.Cu at (333.3, 152.0)
- added R106: 680R, Resistor_SMD:R_0402_1005Metric, F.Cu at (352.3, 152.0)
- added R107: 680R, Resistor_SMD:R_0402_1005Metric, F.Cu at (371.1, 152.0)
- added R108: 680R, Resistor_SMD:R_0402_1005Metric, F.Cu at (390.1, 142.0)
- added R11: 680R, Resistor_SMD:R_0402_1005Metric, F.Cu at (85.1, 57.0)
- added R12: 680R, Resistor_SMD:R_0402_1005Metric, F.Cu at (103.9, 57.0)
- added R13: 680R, Resistor_SMD:R_0402_1005Metric, F.Cu at (123.1, 57.0)
- added R14: 680R, Resistor_SMD:R_0402_1005Metric, F.Cu at (141.8, 57.0)
- added R15: 680R, Resistor_SMD:R_0402_1005Metric, F.Cu at (160.9, 57.0)
- added R16: 680R, Resistor_SMD:R_0402_1005Metric, F.Cu at (180.1, 57.0)
- added R17: 680R, Resistor_SMD:R_0402_1005Metric, F.Cu at (198.8, 57.0)
- added R18: 680R, Resistor_SMD:R_0402_1005Metric, F.Cu at (217.7, 57.0)
- added R19: 680R, Resistor_SMD:R_0402_1005Metric, F.Cu at (236.5, 57.0)
- added R2: 1k, Resistor_SMD:R_0402_1005Metric, F.Cu at (59.1, 38.1)
- added R20: 680R, Resistor_SMD:R_0402_1005Metric, F.Cu at (255.5, 57.0)
- added R21: 680R, Resistor_SMD:R_0402_1005Metric, F.Cu at (275.3, 57.0)
- added R22: 680R, Resistor_SMD:R_0402_1005Metric, F.Cu at (294.7, 57.0)
- added R23: 680R, Resistor_SMD:R_0402_1005Metric, F.Cu at (313.9, 57.0)
- added R24: 680R, Resistor_SMD:R_0402_1005Metric, F.Cu at (332.7, 57.0)
- added R25: 680R, Resistor_SMD:R_0402_1005Metric, F.Cu at (351.7, 57.0)
- added R26: 680R, Resistor_SMD:R_0402_1005Metric, F.Cu at (370.9, 57.0)
- added R27: 680R, Resistor_SMD:R_0402_1005Metric, F.Cu at (389.7, 57.0)
- added R28: 680R, Resistor_SMD:R_0402_1005Metric, F.Cu at (46.6, 76.0)
- added R29: 680R, Resistor_SMD:R_0402_1005Metric, F.Cu at (66.4, 76.0)
- added R3: 27.4, Resistor_SMD:R_0402_1005Metric, F.Cu at (60.6, 27.5)
- added R30: 680R, Resistor_SMD:R_0402_1005Metric, F.Cu at (85.3, 76.0)
- added R31: 680R, Resistor_SMD:R_0402_1005Metric, F.Cu at (104.5, 76.0)
- added R32: 680R, Resistor_SMD:R_0402_1005Metric, F.Cu at (123.3, 76.0)
- added R33: 680R, Resistor_SMD:R_0402_1005Metric, F.Cu at (142.2, 76.0)
- added R34: 680R, Resistor_SMD:R_0402_1005Metric, F.Cu at (160.7, 76.0)
- added R35: 680R, Resistor_SMD:R_0402_1005Metric, F.Cu at (180.3, 76.0)
- added R36: 680R, Resistor_SMD:R_0402_1005Metric, F.Cu at (199.3, 76.0)
- added R37: 680R, Resistor_SMD:R_0402_1005Metric, F.Cu at (219.1, 76.0)
- added R38: 680R, Resistor_SMD:R_0402_1005Metric, F.Cu at (237.1, 76.0)
- added R39: 680R, Resistor_SMD:R_0402_1005Metric, F.Cu at (256.0, 76.0)
- added R4: 27.4, Resistor_SMD:R_0402_1005Metric, F.Cu at (60.6, 26.5)
- added R40: 680R, Resistor_SMD:R_0402_1005Metric, F.Cu at (276.4, 76.0)
- added R41: 680R, Resistor_SMD:R_0402_1005Metric, F.Cu at (305.1, 76.0)
- added R42: 680R, Resistor_SMD:R_0402_1005Metric, F.Cu at (333.2, 76.0)
- added R43: 680R, Resistor_SMD:R_0402_1005Metric, F.Cu at (352.2, 76.0)
- added R44: 680R, Resistor_SMD:R_0402_1005Metric, F.Cu at (371.1, 76.0)
- added R45: 680R, Resistor_SMD:R_0402_1005Metric, F.Cu at (389.4, 76.0)
- added R46: 680R, Resistor_SMD:R_0402_1005Metric, F.Cu at (52.0, 95.0)
- added R47: 680R, Resistor_SMD:R_0402_1005Metric, F.Cu at (76.3, 95.0)
- added R48: 680R, Resistor_SMD:R_0402_1005Metric, F.Cu at (95.5, 95.0)
- added R49: 680R, Resistor_SMD:R_0402_1005Metric, F.Cu at (113.9, 95.0)
- added R5: 5.1k, Resistor_SMD:R_0402_1005Metric, F.Cu at (42.5, 23.0)
- added R50: 680R, Resistor_SMD:R_0402_1005Metric, F.Cu at (133.0, 95.0)
- added R51: 680R, Resistor_SMD:R_0402_1005Metric, F.Cu at (151.9, 95.0)
- added R52: 680R, Resistor_SMD:R_0402_1005Metric, F.Cu at (170.2, 95.0)
- added R53: 680R, Resistor_SMD:R_0402_1005Metric, F.Cu at (189.5, 95.0)
- added R54: 680R, Resistor_SMD:R_0402_1005Metric, F.Cu at (209.6, 95.0)
- added R55: 680R, Resistor_SMD:R_0402_1005Metric, F.Cu at (228.6, 95.0)
- added R56: 680R, Resistor_SMD:R_0402_1005Metric, F.Cu at (247.5, 95.0)
- added R57: 680R, Resistor_SMD:R_0402_1005Metric, F.Cu at (266.3, 95.0)
- added R58: 680R, Resistor_SMD:R_0402_1005Metric, F.Cu at (285.3, 95.0)
- added R59: 680R, Resistor_SMD:R_0402_1005Metric, F.Cu at (309.3, 95.0)
- added R6: 5.1k, Resistor_SMD:R_0402_1005Metric, F.Cu at (46.5, 22.5)
- added R60: 680R, Resistor_SMD:R_0402_1005Metric, F.Cu at (333.7, 95.0)
- added R61: 680R, Resistor_SMD:R_0402_1005Metric, F.Cu at (351.9, 95.0)
- added R62: 680R, Resistor_SMD:R_0402_1005Metric, F.Cu at (370.8, 95.0)
- added R63: 680R, Resistor_SMD:R_0402_1005Metric, F.Cu at (54.5, 114.0)
- added R64: 680R, Resistor_SMD:R_0402_1005Metric, F.Cu at (80.4, 114.0)
- added R65: 680R, Resistor_SMD:R_0402_1005Metric, F.Cu at (99.4, 114.0)
- added R66: 680R, Resistor_SMD:R_0402_1005Metric, F.Cu at (118.5, 114.0)
- added R67: 680R, Resistor_SMD:R_0402_1005Metric, F.Cu at (137.5, 114.0)
- added R68: 680R, Resistor_SMD:R_0402_1005Metric, F.Cu at (156.5, 114.0)
- added R69: 680R, Resistor_SMD:R_0402_1005Metric, F.Cu at (175.5, 114.0)
- added R7: 4.7k, Resistor_SMD:R_0402_1005Metric, F.Cu at (63.5, 36.0)
- added R70: 680R, Resistor_SMD:R_0402_1005Metric, F.Cu at (194.5, 114.0)
- added R71: 680R, Resistor_SMD:R_0402_1005Metric, F.Cu at (213.5, 114.0)
- added R72: 680R, Resistor_SMD:R_0402_1005Metric, F.Cu at (232.2, 114.0)
- added R73: 680R, Resistor_SMD:R_0402_1005Metric, F.Cu at (251.3, 114.0)
- added R74: 680R, Resistor_SMD:R_0402_1005Metric, F.Cu at (271.5, 114.0)
- added R75: 680R, Resistor_SMD:R_0402_1005Metric, F.Cu at (303.3, 114.0)
- added R76: 680R, Resistor_SMD:R_0402_1005Metric, F.Cu at (333.5, 114.0)
- added R77: 680R, Resistor_SMD:R_0402_1005Metric, F.Cu at (351.9, 114.0)
- added R78: 680R, Resistor_SMD:R_0402_1005Metric, F.Cu at (371.3, 114.0)
- added R79: 680R, Resistor_SMD:R_0402_1005Metric, F.Cu at (390.5, 105.0)
- added R8: 4.7k, Resistor_SMD:R_0402_1005Metric, F.Cu at (65.5, 36.0)
- added R80: 680R, Resistor_SMD:R_0402_1005Metric, F.Cu at (59.5, 133.0)
- added R81: 680R, Resistor_SMD:R_0402_1005Metric, F.Cu at (90.3, 133.0)
- added R82: 680R, Resistor_SMD:R_0402_1005Metric, F.Cu at (109.5, 133.0)
- added R83: 680R, Resistor_SMD:R_0402_1005Metric, F.Cu at (128.3, 133.0)
- added R84: 680R, Resistor_SMD:R_0402_1005Metric, F.Cu at (147.5, 133.0)
- added R85: 680R, Resistor_SMD:R_0402_1005Metric, F.Cu at (166.7, 133.0)
- added R86: 680R, Resistor_SMD:R_0402_1005Metric, F.Cu at (185.4, 133.0)
- added R87: 680R, Resistor_SMD:R_0402_1005Metric, F.Cu at (204.6, 133.0)
- added R88: 680R, Resistor_SMD:R_0402_1005Metric, F.Cu at (223.5, 133.0)
- added R89: 680R, Resistor_SMD:R_0402_1005Metric, F.Cu at (242.2, 133.0)
- added R9: 680R, Resistor_SMD:R_0402_1005Metric, F.Cu at (47.5, 57.0)
- added R90: 680R, Resistor_SMD:R_0402_1005Metric, F.Cu at (261.3, 133.0)
- added R91: 680R, Resistor_SMD:R_0402_1005Metric, F.Cu at (287.5, 133.0)
- added R92: 680R, Resistor_SMD:R_0402_1005Metric, F.Cu at (314.3, 133.0)
- added R93: 680R, Resistor_SMD:R_0402_1005Metric, F.Cu at (332.5, 133.0)
- added R94: 680R, Resistor_SMD:R_0402_1005Metric, F.Cu at (351.5, 133.0)
- added R95: 680R, Resistor_SMD:R_0402_1005Metric, F.Cu at (371.3, 133.0)
- added R96: 680R, Resistor_SMD:R_0402_1005Metric, F.Cu at (49.1, 152.0)
- added R97: 680R, Resistor_SMD:R_0402_1005Metric, F.Cu at (74.1, 152.2)
- added R98: 680R, Resistor_SMD:R_0402_1005Metric, F.Cu at (97.3, 152.0)
- added R99: 680R, Resistor_SMD:R_0402_1005Metric, F.Cu at (166.9, 152.0)
- added S1: USB BOOT, TS-1187A-B-A-B:SW_TS-1187A-B-A-B, F.Cu at (37.0, 33.1)
- added SW1: Esc, PG151101S11:SW_PG151101S11, F.Cu at (50.0, 50.0)
- added SW10: F9, PG151101S11:SW_PG151101S11, F.Cu at (221.4, 50.0)
- added SW100: Enter, PG151101S11:SW_PG151101S11, F.Cu at (392.9, 135.7)
- added SW11: F10, PG151101S11:SW_PG151101S11, F.Cu at (240.5, 50.0)
- added SW12: F11, PG151101S11:SW_PG151101S11, F.Cu at (259.6, 50.0)
- added SW13: F12, PG151101S11:SW_PG151101S11, F.Cu at (278.6, 50.0)
- added SW14: DEL, PG151101S11:SW_PG151101S11, F.Cu at (297.6, 50.0)
- added SW15: HOME, PG151101S11:SW_PG151101S11, F.Cu at (316.7, 50.0)
- added SW16: END, PG151101S11:SW_PG151101S11, F.Cu at (335.8, 50.0)
- added SW17: PGUP, PG151101S11:SW_PG151101S11, F.Cu at (354.8, 50.0)
- added SW18: PGDN, PG151101S11:SW_PG151101S11, F.Cu at (373.9, 50.0)
- added SW19: INS, PG151101S11:SW_PG151101S11, F.Cu at (392.9, 50.0)
- added SW2: F1, PG151101S11:SW_PG151101S11, F.Cu at (69.0, 50.0)
- added SW20: TILDE, PG151101S11:SW_PG151101S11, F.Cu at (50.0, 69.0)
- added SW21: 1, PG151101S11:SW_PG151101S11, F.Cu at (69.0, 69.0)
- added SW22: 2, PG151101S11:SW_PG151101S11, F.Cu at (88.1, 69.0)
- added SW23: 3, PG151101S11:SW_PG151101S11, F.Cu at (107.2, 69.0)
- added SW24: 4, PG151101S11:SW_PG151101S11, F.Cu at (126.2, 69.0)
- added SW25: 5, PG151101S11:SW_PG151101S11, F.Cu at (145.2, 69.0)
- added SW26: 6, PG151101S11:SW_PG151101S11, F.Cu at (164.3, 69.0)
- added SW27: 7, PG151101S11:SW_PG151101S11, F.Cu at (183.3, 69.0)
- added SW28: 8, PG151101S11:SW_PG151101S11, F.Cu at (202.4, 69.0)
- added SW29: 9, PG151101S11:SW_PG151101S11, F.Cu at (221.4, 69.0)
- added SW3: F2, PG151101S11:SW_PG151101S11, F.Cu at (88.1, 50.0)
- added SW30: 0, PG151101S11:SW_PG151101S11, F.Cu at (240.5, 69.0)
- added SW31: -, PG151101S11:SW_PG151101S11, F.Cu at (259.6, 69.0)
- added SW32: =, PG151101S11:SW_PG151101S11, F.Cu at (278.6, 69.0)
- added SW33: BKSP, PG151101S11:SW_PG151101S11, F.Cu at (307.2, 69.0)
- added SW34: Num, PG151101S11:SW_PG151101S11, F.Cu at (335.8, 69.0)
- added SW35: /, PG151101S11:SW_PG151101S11, F.Cu at (354.8, 69.0)
- added SW36: *, PG151101S11:SW_PG151101S11, F.Cu at (373.9, 69.0)
- added SW37: -, PG151101S11:SW_PG151101S11, F.Cu at (392.9, 69.0)
- added SW38: Tab, PG151101S11:SW_PG151101S11, F.Cu at (54.8, 88.1)
- added SW39: Q, PG151101S11:SW_PG151101S11, F.Cu at (78.6, 88.1)
- added SW4: F3, PG151101S11:SW_PG151101S11, F.Cu at (107.2, 50.0)
- added SW40: W, PG151101S11:SW_PG151101S11, F.Cu at (97.6, 88.1)
- added SW41: E, PG151101S11:SW_PG151101S11, F.Cu at (116.7, 88.1)
- added SW42: R, PG151101S11:SW_PG151101S11, F.Cu at (135.7, 88.1)
- added SW43: T, PG151101S11:SW_PG151101S11, F.Cu at (154.8, 88.1)
- added SW44: Y, PG151101S11:SW_PG151101S11, F.Cu at (173.8, 88.1)
- added SW45: U, PG151101S11:SW_PG151101S11, F.Cu at (192.9, 88.1)
- added SW46: I, PG151101S11:SW_PG151101S11, F.Cu at (211.9, 88.1)
- added SW47: O, PG151101S11:SW_PG151101S11, F.Cu at (231.0, 88.1)
- added SW48: P, PG151101S11:SW_PG151101S11, F.Cu at (250.0, 88.1)
- added SW49: [, PG151101S11:SW_PG151101S11, F.Cu at (269.1, 88.1)
- added SW5: F4, PG151101S11:SW_PG151101S11, F.Cu at (126.2, 50.0)
- added SW50: ], PG151101S11:SW_PG151101S11, F.Cu at (288.1, 88.1)
- added SW51: \, PG151101S11:SW_PG151101S11, F.Cu at (311.9, 88.1)
- added SW52: 7, PG151101S11:SW_PG151101S11, F.Cu at (335.8, 88.1)
- added SW53: 8, PG151101S11:SW_PG151101S11, F.Cu at (354.8, 88.1)
- added SW54: 9, PG151101S11:SW_PG151101S11, F.Cu at (373.9, 88.1)
- added SW55: Caps, PG151101S11:SW_PG151101S11, F.Cu at (57.1, 107.2)
- added SW56: A, PG151101S11:SW_PG151101S11, F.Cu at (83.3, 107.2)
- added SW57: S, PG151101S11:SW_PG151101S11, F.Cu at (102.4, 107.2)
- added SW58: D, PG151101S11:SW_PG151101S11, F.Cu at (121.4, 107.2)
- added SW59: F, PG151101S11:SW_PG151101S11, F.Cu at (140.5, 107.2)
- added SW6: F5, PG151101S11:SW_PG151101S11, F.Cu at (145.2, 50.0)
- added SW60: G, PG151101S11:SW_PG151101S11, F.Cu at (159.5, 107.2)
- added SW61: H, PG151101S11:SW_PG151101S11, F.Cu at (178.6, 107.2)
- added SW62: J, PG151101S11:SW_PG151101S11, F.Cu at (197.6, 107.2)
- added SW63: K, PG151101S11:SW_PG151101S11, F.Cu at (216.7, 107.2)
- added SW64: L, PG151101S11:SW_PG151101S11, F.Cu at (235.7, 107.2)
- added SW65: ;, PG151101S11:SW_PG151101S11, F.Cu at (254.8, 107.2)
- added SW66: ", PG151101S11:SW_PG151101S11, F.Cu at (273.8, 107.2)
- added SW67: Enter, PG151101S11:SW_PG151101S11, F.Cu at (305.9, 107.2)
- added SW68: 4, PG151101S11:SW_PG151101S11, F.Cu at (335.8, 107.2)
- added SW69: 5, PG151101S11:SW_PG151101S11, F.Cu at (354.8, 107.2)
- added SW7: F6, PG151101S11:SW_PG151101S11, F.Cu at (164.3, 50.0)
- added SW70: 6, PG151101S11:SW_PG151101S11, F.Cu at (373.9, 107.2)
- added SW71: +, PG151101S11:SW_PG151101S11, F.Cu at (392.9, 97.6)
- added SW72: Shift, PG151101S11:SW_PG151101S11, F.Cu at (61.9, 126.2)
- added SW73: Z, PG151101S11:SW_PG151101S11, F.Cu at (92.9, 126.2)
- added SW74: X, PG151101S11:SW_PG151101S11, F.Cu at (111.9, 126.2)
- added SW75: C, PG151101S11:SW_PG151101S11, F.Cu at (131.0, 126.2)
- added SW76: V, PG151101S11:SW_PG151101S11, F.Cu at (150.0, 126.2)
- added SW77: B, PG151101S11:SW_PG151101S11, F.Cu at (169.1, 126.2)
- added SW78: N, PG151101S11:SW_PG151101S11, F.Cu at (188.1, 126.2)
- added SW79: M, PG151101S11:SW_PG151101S11, F.Cu at (207.2, 126.2)
- added SW8: F7, PG151101S11:SW_PG151101S11, F.Cu at (183.3, 50.0)
- added SW80: <, PG151101S11:SW_PG151101S11, F.Cu at (226.2, 126.2)
- added SW81: >, PG151101S11:SW_PG151101S11, F.Cu at (245.3, 126.2)
- added SW82: /, PG151101S11:SW_PG151101S11, F.Cu at (264.3, 126.2)
- added SW83: Shift, PG151101S11:SW_PG151101S11, F.Cu at (290.5, 126.2)
- added SW84: Up, PG151101S11:SW_PG151101S11, F.Cu at (316.7, 126.2)
- added SW85: 1, PG151101S11:SW_PG151101S11, F.Cu at (335.8, 126.2)
- added SW86: 2, PG151101S11:SW_PG151101S11, F.Cu at (354.8, 126.2)
- added SW87: 3, PG151101S11:SW_PG151101S11, F.Cu at (373.9, 126.2)
- added SW88: Ctrl, PG151101S11:SW_PG151101S11, F.Cu at (52.4, 145.2)
- added SW89: Win, PG151101S11:SW_PG151101S11, F.Cu at (76.2, 145.2)
- added SW9: F8, PG151101S11:SW_PG151101S11, F.Cu at (202.4, 50.0)
- added SW90: Alt, PG151101S11:SW_PG151101S11, F.Cu at (100.0, 145.2)
- added SW91: Space, PG151101S11:SW_PG151101S11, F.Cu at (170.3, 145.2)
- added SW92: Fn, PG151101S11:SW_PG151101S11, F.Cu at (240.5, 145.2)
- added SW93: M1, PG151101S11:SW_PG151101S11, F.Cu at (259.6, 145.2)
- added SW94: M2, PG151101S11:SW_PG151101S11, F.Cu at (278.6, 145.2)
- added SW95: Left, PG151101S11:SW_PG151101S11, F.Cu at (297.6, 145.2)
- added SW96: Down, PG151101S11:SW_PG151101S11, F.Cu at (316.7, 145.2)
- added SW97: Right, PG151101S11:SW_PG151101S11, F.Cu at (335.8, 145.2)
- added SW98: 0, PG151101S11:SW_PG151101S11, F.Cu at (354.8, 145.2)
- added SW99: ., PG151101S11:SW_PG151101S11, F.Cu at (373.9, 145.2)
- added U1: RP2040, Package_DFN_QFN:QFN-56-1EP_7x7mm_P0.4mm_EP3.2x3.2mm, F.Cu at (66.2, 28.2)
- added U2: NCP1117-3.3_SOT223, Package_TO_SOT_SMD:SOT-223-3_TabPin2, F.Cu at (44.6, 33.0)
- added U3: W25Q128JVS, W25Q128JVSIQ:SOIC127P790X216-8N, F.Cu at (55.4, 34.5)
- added U4: ABM8-272-T3, ABM8:XTAL_ABM8-272-T3, F.Cu at (85.2, 20.0)
- added U5: MCP23017 1, Package_DFN_QFN:QFN-28-1EP_6x6mm_P0.65mm_EP4.25x4.25mm, F.Cu at (150.0, 29.9)
- added U6: MCP23017 2, Package_DFN_QFN:QFN-28-1EP_6x6mm_P0.65mm_EP4.25x4.25mm, F.Cu at (364.5, 29.4)
- added U7: IRLML6344TRPBF, IRLML6344TRPBF:SOT95P240X112-3N, F.Cu at (33.0, 39.0)
Routing:
- net Net-(U7-D): track 0.00 -> 2606.4 mm, vias 0 -> 4
- net +5V: track 0.00 -> 2496.0 mm, vias 0 -> 24
- net VREG: track 0.00 -> 647.3 mm, vias 0 -> 11
- net SPI_MOSI: track 0.00 -> 579.8 mm, vias 0 -> 2
- net SPI_MISO: track 0.00 -> 578.7 mm, vias 0 -> 2
- net SPI_SCK: track 0.00 -> 573.2 mm, vias 0 -> 2
- net TOUCH_INT: track 0.00 -> 509.4 mm, vias 0 -> 2
- net SPI_TOUCH_CS: track 0.00 -> 502.9 mm, vias 0 -> 2
- net R6: track 0.00 -> 500.3 mm, vias 0 -> 24
- net TOUCH_LED: track 0.00 -> 496.6 mm, vias 0 -> 2
- net DISPLAY_DC: track 0.00 -> 489.7 mm, vias 0 -> 2
- net SPI_DISPLAY_CS: track 0.00 -> 488.7 mm, vias 0 -> 2
- net R5: track 0.00 -> 472.8 mm, vias 0 -> 32
- net R4: track 0.00 -> 452.6 mm, vias 0 -> 32
- net R3: track 0.00 -> 440.2 mm, vias 0 -> 34
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- added copper zone on B.Cu, net GND
Other:
- board outline added: 440 x 150 mm

Commit message: yeah, just everything
Parts:
- added R109: PTA3043-2010CIB103, PTA3043-2010CIB103:TRIM_PTA3043-2010CIB103, F.Cu at (432.9, 54.4)
- added R110: PTA3043-2010CIB103, PTA3043-2010CIB103:TRIM_PTA3043-2010CIB103, F.Cu at (432.9, 67.0)
- added REF**: MountingHole_2.2mm_M2, MountingHole:MountingHole_2.2mm_M2, F.Cu at (24.0, 160.0)
- added REF**: MountingHole_2.2mm_M2, MountingHole:MountingHole_2.2mm_M2, F.Cu at (456.0, 18.0)
- added REF**: MountingHole_2.2mm_M2, MountingHole:MountingHole_2.2mm_M2, F.Cu at (455.0, 159.0)
- added REF**: MountingHole_2.2mm_M2, MountingHole:MountingHole_2.2mm_M2, F.Cu at (24.0, 18.0)
- added SW101: RotaryEncoder, EC10E1220501:TRIM_EC10E1220501, F.Cu at (430.0, 35.4)
- J1, J2: moved to B.Cu
- SW1, SW10, SW11, SW12, SW13, SW14, SW15, SW16, SW17, SW18, SW19, SW2, SW20, SW21, SW22, SW23, SW24, SW25, SW26, SW27, SW28, SW29, SW3, SW30, SW31, SW32, SW34, SW35, SW36, SW37, SW39, SW4, SW40, SW41, SW42, SW43, SW44, SW45, SW46, SW47, SW48, SW49, SW5, SW50, SW52, SW53, SW54, SW56, SW57, SW58, SW59, SW6, SW60, SW61, SW62, SW63, SW64, SW65, SW66, SW68, SW69, SW7, SW70, SW73, SW74, SW75, SW76, SW77, SW78, SW79, SW8, SW80, SW81, SW82, SW84, SW85, SW86, SW87, SW9, SW92, SW93, SW94, SW95, SW96, SW97, SW98, SW99: footprint PG151101S11:SW_PG151101S11 -> MX_Hotswap:MX-Hotswap-1U; moved to B.Cu
- SW100, SW71: footprint PG151101S11:SW_PG151101S11 -> MX_Hotswap:MX-Hotswap-2U-Vertical; moved to B.Cu
- SW33: footprint PG151101S11:SW_PG151101S11 -> MX_Hotswap:MX-Hotswap-2U; moved to B.Cu
- SW38, SW51: footprint PG151101S11:SW_PG151101S11 -> MX_Hotswap:MX-Hotswap-1.5U; moved to B.Cu
- SW55, SW83: footprint PG151101S11:SW_PG151101S11 -> MX_Hotswap:MX-Hotswap-1.75U; moved to B.Cu
- SW67, SW72: footprint PG151101S11:SW_PG151101S11 -> MX_Hotswap:MX-Hotswap-2.25U; moved to B.Cu
- SW88, SW89, SW90: footprint PG151101S11:SW_PG151101S11 -> MX_Hotswap:MX-Hotswap-1.25U; moved to B.Cu
- SW91: footprint PG151101S11:SW_PG151101S11 -> MX_Hotswap:MX-Hotswap-6.25U; moved to B.Cu
- moved J1 30.1 mm to (31.0, -5.30)
- moved J2 30.0 mm to (43.1, -13.7), turned to 0 degrees
- moved R5 27.5 mm to (41.3, -4.51)
- moved R6 27.5 mm to (46.1, -5.00)
- turned SW1 to 180 degrees
- turned SW10 to 180 degrees
- turned SW100 to 180 degrees
- turned SW11 to 180 degrees
- turned SW12 to 180 degrees
- turned SW13 to 180 degrees
- turned SW14 to 180 degrees
- turned SW15 to 180 degrees
- turned SW16 to 180 degrees
- turned SW17 to 180 degrees
- turned SW18 to 180 degrees
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Connections:
- U1 pad 15: EA -> unconnected-(U1-GPIO12-Pad15)
- U1 pad 16: EB -> unconnected-(U1-GPIO13-Pad16)
- U1 pad 17: POT_1 -> unconnected-(U1-GPIO14-Pad17)
- U1 pad 18: POT_2 -> unconnected-(U1-GPIO15-Pad18)
- U6 pad 2: unconnected-(U6-GPB5-Pad2) -> EA
- U6 pad 23: unconnected-(U6-GPA6-Pad23) -> POT_2
- U6 pad 3: unconnected-(U6-GPB6-Pad3) -> EB
- U6 pad 4: unconnected-(U6-GPB7-Pad4) -> POT_1
Routing:
- net VREG: track 647.3 -> 777.2 mm
- net POT_1: track 0.00 -> 82.5 mm, vias 0 -> 3
- net EB: track 0.00 -> 78.1 mm, vias 0 -> 6
- net EA: track 0.00 -> 75.0 mm, vias 0 -> 6
- net POT_2: track 0.00 -> 72.4 mm, vias 0 -> 4
- net GND: track 237.8 -> 204.3 mm, vias 11 -> 12
- net Net-(U7-D): track 2606.4 -> 2592.7 mm, vias 4 -> 2
- net C15: track 174.4 -> 187.6 mm, vias 0 -> 1
- net +5V: track 2496.0 -> 2507.1 mm, vias 24 -> 45
- net C13: track 260.2 -> 249.6 mm, vias 0 -> 1
- net C12: track 239.7 -> 231.3 mm, vias 0 -> 1
- net C10: track 177.3 -> 169.2 mm, vias 0 -> 1
- net C9: track 157.2 -> 149.1 mm, vias 0 -> 1
- net C8: track 137.3 -> 129.3 mm, vias 0 -> 1
- net Net-(D71-A): track 3.21 -> 11.1 mm, vias 0 -> 1
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Other:
- board size 440 x 150 mm -> 440 x 180 mm
