File: pcb/main_board/main_board.kicad_pcb (KiCad board)
At the start: 2 copper layers, 440 x 137.2 mm, 419 parts, among them J1 Conn_02x30_Odd_Even, J3 Touchscreen, J4 Touchscreen, M1 Motor_Servo, M10 Motor_Servo, M2 Motor_Servo, M3 Motor_Servo, M4 Motor_Servo, M5 Motor_Servo, M6 Motor_Servo, M7 Motor_Servo, M8 Motor_Servo, M9 Motor_Servo, SW1 Esc, SW10 F9, SW100 Enter, SW101 RotaryEncoder, SW11 F10, SW12 F11, SW13 F12, SW14 DEL, SW15 HOME, SW16 END, SW17 PGUP, SW18 PGDN, SW19 INS, SW2 F1, SW20 TILDE, SW21 1, SW22 2, SW23 3, SW24 4, SW25 5, SW26 6, SW27 7, SW28 8, SW29 9, SW3 F2, SW30 0, SW31 -, SW32 =, SW33 BKSP, SW34 Num, SW35 /, SW36 *, SW37 -, SW38 Tab, SW39 Q, SW4 F3, SW40 W, SW41 E, SW42 R, SW43 T, SW44 Y, SW45 U, SW46 I, SW47 O, SW48 P, SW49 [, SW5 F4, SW50 ], SW51 \, SW52 7, SW53 8, SW54 9, SW55 Caps, SW56 A, SW57 S, SW58 D, SW59 F, SW6 F5, SW60 G, SW61 H, SW62 J, SW63 K, SW64 L, SW65 ;, SW66 ", SW67 Enter, SW68 4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

Commit message: add renders and finish and export case
Parts:
- added REF**: MountingHole_2.2mm_M2, MountingHole:MountingHole_2.2mm_M2, F.Cu at (24.0, 31.2)
- added REF**: MountingHole_2.2mm_M2, MountingHole:MountingHole_2.2mm_M2, F.Cu at (24.0, 95.6)
- added REF**: MountingHole_2.2mm_M2, MountingHole:MountingHole_2.2mm_M2, F.Cu at (455.0, 95.6)
- added REF**: MountingHole_2.2mm_M2, MountingHole:MountingHole_2.2mm_M2, F.Cu at (456.0, 31.2)
- moved J1 2.47 mm to (71.5, 33.3)
- moved REF** 1.41 mm to (456.0, 160.0)
Routing:
- net GND: track 198.1 -> 222.2 mm, vias 19 -> 23
- net +3V3: track 831.0 -> 836.0 mm
- net C12: track 314.8 -> 311.0 mm, vias 1 -> 2
- net C13: track 331.7 -> 328.1 mm, vias 1 -> 2
- net C15: track 383.5 -> 380.0 mm, vias 1 -> 2
- net C14: track 381.2 -> 377.7 mm, vias 1 -> 2
- net C16: track 385.5 -> 382.0 mm, vias 1 -> 2
- net C17: track 406.3 -> 402.8 mm, vias 1 -> 2
- net C18: track 427.2 -> 423.7 mm, vias 1 -> 2
- net C19: track 443.4 -> 439.9 mm, vias 1 -> 2
- net SERVO_8: track 255.8 -> 258.3 mm
- net SERVO_7: track 224.6 -> 227.1 mm
- net SERVO_9: track 287.0 -> 289.5 mm
- net SERVO_6: track 193.4 -> 195.9 mm
- net SERVO_5: track 162.2 -> 164.7 mm
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Other:
- outline, holes or cut-outs redrawn
